Commit message: flip LiDAR joint + link around
in ``x3_peripherals.xacro``:
- rotate visual to be forward facing
- rotate joint to be forward facing

in ``robot.launch.py``:
- switch scan mode to standard
- set flip x axis flag to true

File: src/x3_description/urdf/x3_peripherals.xacro (robot description, xacro)
@@ -5,9 +5,9 @@
     <link name = "${prefix}_lidar_link">
         <visual>
-            <origin xyz = "0 0 0" rpy = "1.570796 0 -1.570796"/>
+            <origin xyz = "0 0 0" rpy = "1.570796 0 1.570796"/>
             <geometry>
                 <mesh filename = "package://x3_description/meshes/lidar.STL" scale = "0.001 0.001 0.001"/>
             </geometry>
-            <material name = "black"/>
+            <material name = "blue"/>
         </visual>
         <collision>
@@ -28,5 +28,5 @@
     <!-- lidar to chassis joint -->
     <joint name = "${prefix}_lidar_joint" type = "fixed">
-        <origin xyz = "0.0405 5.25826986680105E-05 0.08285" rpy = "0 0 3.141592"/>         <!-- z is 0.08285 to chassis_link, 0.154 if from base_link -->
+        <origin xyz = "0.0405 5.25826986680105E-05 0.08285" rpy = "0 0 0"/>         <!-- z is 0.08285 to chassis_link, 0.154 if from base_link -->
         <parent link = "${prefix}_chassis_link"/>
         <child link = "${prefix}_lidar_link"/>

Commit message: return to backward facing LiDAR joint
in ``robot_launch.py``:
- commented out ``flip_x_axis`` param

in ``x3_peripherals.xacro``:
- flipped joint to be backwards
- flipped visual to be forward facing relative to new joint orientation

in ``policy_node.py``:
- increased obstacle tolerance
- commented out a debug print
- removed antennae mask

these changes were done after observing that the DRL policy broke when the joint was flipped, and I don't want to debug why it doesn't work

File: src/x3_description/urdf/x3_peripherals.xacro (robot description, xacro)
@@ -5,5 +5,5 @@
     <link name = "${prefix}_lidar_link">
         <visual>
-            <origin xyz = "0 0 0" rpy = "1.570796 0 1.570796"/>
+            <origin xyz = "0 0 0" rpy = "1.570796 0 -1.570796"/>
             <geometry>
                 <mesh filename = "package://x3_description/meshes/lidar.STL" scale = "0.001 0.001 0.001"/>
@@ -28,5 +28,5 @@
     <!-- lidar to chassis joint -->
     <joint name = "${prefix}_lidar_joint" type = "fixed">
-        <origin xyz = "0.0405 5.25826986680105E-05 0.08285" rpy = "0 0 0"/>         <!-- z is 0.08285 to chassis_link, 0.154 if from base_link -->
+        <origin xyz = "0.0405 5.25826986680105E-05 0.08285" rpy = "0 0 3.141592"/>         <!-- z is 0.08285 to chassis_link, 0.154 if from base_link -->
         <parent link = "${prefix}_chassis_link"/>
         <child link = "${prefix}_lidar_link"/>

Commit message: make LiDAR visual black

File: src/x3_description/urdf/x3_peripherals.xacro (robot description, xacro)
@@ -9,5 +9,5 @@
                 <mesh filename = "package://x3_description/meshes/lidar.STL" scale = "0.001 0.001 0.001"/>
             </geometry>
-            <material name = "blue"/>
+            <material name = "black"/>
         </visual>
         <collision>

Commit message: switch to forward facing LiDAR joint and filter back of scans
in ``x3_peripherals.xacro``:
- switch joint to be forward facing

in ``lidar_rear_mask.py``:
- initial commit on a new node used to mask out the rear portion of the LiDAR scan data. this is done so that the phantom traces in the LiDAR do not ruin the LiDAR odometry calculation

in ``setup.py``:
- add entry point for ``lidar_rear_mask.py``

in ``odom.launch.py``:
- switch to using new filtered LiDAR scan topic

in ``robot.launch.py``:
- flipped the x axis on the LiDAR node to reflect forward facing joint
- added launching of rear mask node

in ``policy_node.py``:
- switch lidar subscriber to subscribe to filtered scan topic
- adjust ``lidar_callback()`` method to work with forward facing joint
-  remove index masking and just use blanket distance mask

File: src/x3_description/urdf/x3_peripherals.xacro (robot description, xacro)
@@ -5,5 +5,5 @@
     <link name = "${prefix}_lidar_link">
         <visual>
-            <origin xyz = "0 0 0" rpy = "1.570796 0 -1.570796"/>
+            <origin xyz = "0 0 0" rpy = "1.570796 0 1.570796"/>
             <geometry>
                 <mesh filename = "package://x3_description/meshes/lidar.STL" scale = "0.001 0.001 0.001"/>
@@ -28,5 +28,5 @@
     <!-- lidar to chassis joint -->
     <joint name = "${prefix}_lidar_joint" type = "fixed">
-        <origin xyz = "0.0405 5.25826986680105E-05 0.08285" rpy = "0 0 3.141592"/>         <!-- z is 0.08285 to chassis_link, 0.154 if from base_link -->
+        <origin xyz = "0.0405 5.25826986680105E-05 0.08285" rpy = "0 0 0"/>         <!-- z is 0.08285 to chassis_link, 0.154 if from base_link -->
         <parent link = "${prefix}_chassis_link"/>
         <child link = "${prefix}_lidar_link"/>
